Commit message: URDF from gpt that needs fix

File: urdf/UR16e_gpt.urdf (robot description, URDF)
Before this commit: robot eSeries_UR16e_15012020_URDF_ONLY, 8 links, 7 joints
Links:
- removed link Shoulder1
- added link Shoulder, mass 7.369; collision mesh filename=meshes/Link1.STL; visual mesh filename=meshes/Link1.STL
Joints:
- joint J1: child Shoulder1 -> Shoulder
- joint J2: parent Shoulder1 -> Shoulder
