Commit message: Fixed urdf and meshes

File: urdf/UR16e_fixed.urdf (robot description, URDF)
Before this commit: robot eSeries_UR16e_15012020_URDF_ONLY, 8 links, 7 joints
Links:
- link Elbow: geometry collision mesh filename=meshes/elbow.stl; visual mesh filename=meshes/elbow.stl
- link EndEffector: geometry collision mesh filename=meshes/end_effector.stl; visual mesh filename=meshes/end_effector.stl
- link Shoulder1: geometry collision mesh filename=meshes/shoulder1.stl; visual mesh filename=meshes/shoulder1.stl
- link Shoulder2: geometry collision mesh filename=meshes/shoulder2.stl; visual mesh filename=meshes/shoulder2.stl
- link Wrist1: geometry collision mesh filename=meshes/wrist1.stl; visual mesh filename=meshes/wrist1.stl
- link Wrist2: geometry collision mesh filename=meshes/wrist2.stl; visual mesh filename=meshes/wrist2.stl
- link Wrist3: geometry collision mesh filename=meshes/wrist3.stl; visual mesh filename=meshes/wrist3.stl
- link base_link: geometry collision mesh filename=meshes/base_link.stl; visual mesh filename=meshes/base_link.stl
Joints:
- joint J1: origin xyz=0 0 0.0993 rpy=1.5708 0 0 -> xyz=0 0 0 rpy=0 0 0
- joint J2: origin xyz=0 0.0814 0.0946 rpy=0 0 1.5708 -> xyz=0 0 0 rpy=0 0 0
- joint J3: origin xyz=0 0.4784 0 rpy=0 0 0 -> xyz=0 0 0 rpy=0 0 0
- joint J4: origin xyz=0 0.36 0 rpy=0 0 1.5707963267949 -> xyz=0 0 0 rpy=0 0 0
- joint J5: limit lower=-1.57 upper=1.57 effort=0 velocity=3.141 -> lower=-6.28 upper=6.28 effort=0 velocity=3.141; origin xyz=0 0.00334216106109189 0.0795500000000001 rpy=0 0 0 -> xyz=0 0 0 rpy=0 0 0
