Commit message: Fixed inverse kinematics coordinates, need collision

File: urdf/ur16e_final.urdf (robot description, URDF)
Before this commit: robot ur16e_robot, 11 links, 10 joints
Links:
- link tool0: geometry collision cylinder length=.4 radius=.2; visual cylinder length=.4 radius=.2
Joints:
- joint shoulder_lift_joint: origin xyz=0 0 0 rpy=1.570796327 1.57 0 -> xyz=0 0 0 rpy=1.570796327 0 0
- joint wrist_1_joint: origin xyz=-0.36 0 0.17415 rpy=0 0 -1.57 -> xyz=-0.36 0 0.17415 rpy=0 0 0
