Commit message: Cleanup and prepare for final demo

File: URandPyBullet/urdf/ur16e_final.urdf (robot description, URDF)
Before this commit: robot ur16e_robot, 11 links, 10 joints
Links:
- link base_link: mass None -> 1.0
- link tool0: mass None -> 0.01; geometry collision cylinder length=.2 radius=.06; visual cylinder length=.2 radius=.06
Joints:
- joint shoulder_lift_joint: limit lower=-6.283185307179586 upper=6.283185307179586 effort=330.0 velocity=2.0943951023931953 -> lower=-3.14159265359 upper=3.14159265359 effort=330.0 velocity=2.0943951023931953
- joint shoulder_pan_joint: limit lower=-6.283185307179586 upper=6.283185307179586 effort=330.0 velocity=2.0943951023931953 -> lower=-3.14159265359 upper=3.14159265359 effort=330.0 velocity=2.0943951023931953
- joint wrist_1_joint: limit lower=-6.283185307179586 upper=6.283185307179586 effort=56.0 velocity=3.141592653589793 -> lower=-3.14159265359 upper=3.14159265359 effort=56.0 velocity=3.141592653589793
- joint wrist_2_joint: limit lower=-6.283185307179586 upper=6.283185307179586 effort=56.0 velocity=3.141592653589793 -> lower=-3.14159265359 upper=3.14159265359 effort=56.0 velocity=3.141592653589793
- joint wrist_3_joint: limit lower=-6.283185307179586 upper=6.283185307179586 effort=56.0 velocity=3.141592653589793 -> lower=-3.14159265359 upper=3.14159265359 effort=56.0 velocity=3.141592653589793

Commit message: Tried to make IK work with robot, end effector is wrong orientation

File: URandPyBullet/urdf/ur16e_final.urdf (robot description, URDF)
Before this commit: robot ur16e_robot, 11 links, 10 joints
Links:
- removed link flange
- removed link tool0
- link base_link: mass 1.0 -> None
Joints:
- removed joint flange-tool0
- removed joint wrist_3-flange
- joint elbow_joint: limit lower=-3.141592653589793 upper=3.141592653589793 effort=150.0 velocity=3.141592653589793 -> lower=-6.28 upper=6.28 effort=150.0 velocity=3.141592653589793
- joint shoulder_lift_joint: limit lower=-3.14159265359 upper=3.14159265359 effort=330.0 velocity=2.0943951023931953 -> lower=-6.28 upper=6.28 effort=330.0 velocity=2.0943951023931953
- joint shoulder_pan_joint: limit lower=-3.14159265359 upper=3.14159265359 effort=330.0 velocity=2.0943951023931953 -> lower=-6.28 upper=6.28 effort=330.0 velocity=2.0943951023931953
- joint wrist_1_joint: limit lower=-3.14159265359 upper=3.14159265359 effort=56.0 velocity=3.141592653589793 -> lower=-6.28 upper=6.28 effort=56.0 velocity=3.141592653589793
- joint wrist_2_joint: limit lower=-3.14159265359 upper=3.14159265359 effort=56.0 velocity=3.141592653589793 -> lower=-6.28 upper=6.28 effort=56.0 velocity=3.141592653589793
- joint wrist_3_joint: limit lower=-3.14159265359 upper=3.14159265359 effort=56.0 velocity=3.141592653589793 -> lower=-6.28 upper=6.28 effort=56.0 velocity=3.141592653589793

File: urdf/ur16e_final.urdf (robot description, URDF)
Before this commit: robot ur16e_robot, 11 links, 10 joints
Links:
- removed link flange
- removed link tool0
Joints:
- removed joint flange-tool0
- removed joint wrist_3-flange
- joint shoulder_lift_joint: limit lower=-6.283185307179586 upper=6.283185307179586 effort=330.0 velocity=2.0943951023931953 -> lower=-3.141592653589793 upper=3.141592653589793 effort=330.0 velocity=2.0943951023931953
- joint shoulder_pan_joint: limit lower=-6.283185307179586 upper=6.283185307179586 effort=330.0 velocity=2.0943951023931953 -> lower=-3.141592653589793 upper=3.141592653589793 effort=330.0 velocity=2.0943951023931953
- joint wrist_1_joint: limit lower=-6.283185307179586 upper=6.283185307179586 effort=56.0 velocity=3.141592653589793 -> lower=-3.141592653589793 upper=3.141592653589793 effort=56.0 velocity=3.141592653589793
- joint wrist_2_joint: limit lower=-6.283185307179586 upper=6.283185307179586 effort=56.0 velocity=3.141592653589793 -> lower=-3.141592653589793 upper=3.141592653589793 effort=56.0 velocity=3.141592653589793
- joint wrist_3_joint: limit lower=-6.283185307179586 upper=6.283185307179586 effort=56.0 velocity=3.141592653589793 -> lower=-3.141592653589793 upper=3.141592653589793 effort=56.0 velocity=3.141592653589793
